Commit message: New code from Gabirell adapted to my needs

File: yumi_description/urdf/yumi.urdf (robot description, URDF)
Before this commit: robot yumi, 22 links, 21 joints
Links:
- added link ftsensor_l, mass 0.2; collision mesh filename=package://yumi_description/meshes/gripper/coarse/forcetourq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; visual mesh filename=package://yumi_description/meshes/gripper/forcetourqe.stl
Joints:
- added joint ftsensor_l_joint: type fixed, parent ftsensor_l, child gripper_l_base, origin xyz=0 0 0.006 rpy=0 0 3.1415926536
- joint yumi_link_7_l_joint: child gripper_l_base -> ftsensor_l; origin xyz=0 0 0.007 rpy=0 0 3.14159265359 -> xyz=0 0 0.0274 rpy=0 0 -3.1415926536
